File: design/RP2350_80QFN_minimal.kicad_sch (KiCad schematic)
At the start: 49 parts, among them J1 USB_B_Micro, J2 Conn_02x26_Odd_Even, J3 Conn_02x26_Odd_Even, J4 SM03B-SRSS-TB, SW1 SW_Push, SW2 SW_Push, U1 RP2350_80QFN, U2 NCP1117-3.3_SOT223, U3 W25Q128JVS, U4 DNF, Y1 ABM8-272-T3

Commit message: stage0: PWR_FLAG on +1V1/VREG_AVDD, re-link W25Q128JVS footprint to KiCad10 name
Parts:
- U3, U4: footprint Package_SO:SOIC-8_5.23x5.23mm_P1.27mm -> Package_SO:SOIC-8_5.3x5.3mm_P1.27mm
Changed lines of the file:
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@@
       (effects (font (size 1.27 1.27)))
     )
-    (property "Footprint" "Package_SO:SOIC-8_5.23x5.23mm_P1.27mm" (at 67.31 127.635 0)
+    (property "Footprint" "Package_SO:SOIC-8_5.3x5.3mm_P1.27mm" (at 67.31 127.635 0)
       (effects (font (size 1.27 1.27)) hide)
     )
@@
     )
   )
+  (symbol (lib_id "power:PWR_FLAG") (at 119.38 101.6 0) (unit 1)
+    (in_bom yes) (on_board yes) (dnp no)
+    (property "Reference" "#FLG01" (at 119.38 99.695 0)
+      (effects (font (size 1.27 1.27)) hide)
+    )
+    (property "Value" "PWR_FLAG" (at 119.38 97.79 0)
+      (effects (font (size 1.27 1.27)))
+    )
+    (property "Footprint" "" (at 119.38 101.6 0)
+      (effects (font (size 1.27 1.27)) hide)
+    )
+    (property "Datasheet" "" (at 119.38 101.6 0)
+      (effects (font (size 1.27 1.27)) hide)
+    )
+    (pin "1")
+    (instances
+      (project "RP2350_80QFN_minimal"
+        (path "/94683f5c-9cd9-448e-be96-9792537b5cb8"
+          (reference "#FLG01") (unit 1)
+        )
+      )
+    )
+  )
+  (symbol (lib_id "power:PWR_FLAG") (at 153.67 90.17 0) (unit 1)
+    (in_bom yes) (on_board yes) (dnp no)
+    (property "Reference" "#FLG02" (at 153.67 88.265 0)
+      (effects (font (size 1.27 1.27)) hide)
+    )
+    (property "Value" "PWR_FLAG" (at 153.67 86.36 0)
+      (effects (font (size 1.27 1.27)))
+    )
+    (property "Footprint" "" (at 153.67 90.17 0)
+      (effects (font (size 1.27 1.27)) hide)
+    )
+    (property "Datasheet" "" (at 153.67 90.17 0)
+      (effects (font (size 1.27 1.27)) hide)
+    )
+    (pin "1")
+    (instances
+      (project "RP2350_80QFN_minimal"
+        (path "/94683f5c-9cd9-448e-be96-9792537b5cb8"
+          (reference "#FLG02") (unit 1)
+        )
+      )
+    )
+  )
   (symbol (lib_id "Switch:SW_Push") (at 133.35 165.1 0) (unit 1)
     (in_bom yes) (on_board yes) (dnp no) (fields_autoplaced)
@@
       (effects (font (size 1.27 1.27)))
     )
-    (property "Footprint" "Package_SO:SOIC-8_5.23x5.23mm_P1.27mm" (at 68.58 186.69 0)
-      (effects (font (size 1.27 1.27)) hide)
-    )
+    (property "Footprint" "Package_SO:SOIC-8_5.3x5.3mm_P1.27mm" (at 68.58 186.69 0)
+      (effects (font (size 1.27 1.27)) hide)
+    )

Commit message: stage1: MPN/LCSC population + datasheet corpus (G1 prep)
Parts:
- C1, C19, C5: LCSC (none) -> C15850; MPN (none) -> CL21A106KAYNNNE
- C10, C6, C7, C9: LCSC (none) -> C23733; MPN (none) -> CL05A475MP5NRNC
- C11, C12, C13, C14, C15, C16, C17, C18, C2, C20, C21, C8: LCSC (none) -> C1525; MPN (none) -> CL05B104KO5NNNC
- C3, C4: LCSC (none) -> C1548; MPN (none) -> 0402CG150J500NT
- J1: LCSC (none) -> C428495; MPN (none) -> 10103594-0001LF
- J2, J3: LCSC (none) -> C725898; MPN (none) -> X6521WV-2x26H-C60D30
- J4: LCSC (none) -> C160403; MPN (none) -> SM03B-SRSS-TB(LF)(SN)
- L1: LCSC (none) -> C42411119; MPN (none) -> AOTA-B201610S3R3-101-T
- R10: LCSC (none) -> C17168; MPN (none) -> 0402WGF0000TCE
- R2, R4, R6: LCSC (none) -> C11702; MPN (none) -> 0402WGF1001TCE
- R3: LCSC (none) -> C25105; MPN (none) -> 0402WGF330JTCE
- R7, R8: LCSC (none) -> C25100; MPN (none) -> 0402WGF270JTCE
- SW1, SW2: LCSC (none) -> C139797; MPN (none) -> SKRPACE010
- U1: LCSC (none) -> C9900208890; MPN (none) -> RP2350B A4
- U2: LCSC (none) -> C26537; MPN (none) -> NCP1117ST33T3G
- U3: LCSC (none) -> C97521; MPN (none) -> W25Q128JVSIQ
- Y1: LCSC (none) -> C20625731; MPN (none) -> ABM8-272-T3
